File: hd44780_tutorial.kicad_pcb (KiCad board)
At the start: 2 copper layers, 157.2 x 83.5 mm, 30 parts, among them J1 LCD_2004_PinSocket_1x16_P2.54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, J2 USB4105-GF-A, SW1 REG SELECT, SW2 ENABLE, SW3 DS02C-254-1L-08BE

Commit message: Revert "Tried a new USB-C port and hate it. Prfeparing to revert to get rid of it."
This reverts commit 31f363ccd091cdbcf9bc00afb548c8c72483716e.
Parts:
- removed D5: RED, LED_THT:LED_D3.0mm
- removed R4: 470, Resistor_THT:R_Axial_DIN0207_L6.3mm_D2.5mm_P7.62mm_Horizontal
- removed RN2: 1KΩ, footprints:R_Array_SIP9
- added D4: RED, LED_THT:LED_D3.0mm, F.Cu at (214.1, 82.0)
- added R6: 330Ω, Resistor_THT:R_Axial_DIN0207_L6.3mm_D2.5mm_P7.62mm_Horizontal, F.Cu at (207.4, 78.4)
- added REF**: OSHW-Logo2_14.6x12mm_SilkScreen, Symbol:OSHW-Logo2_14.6x12mm_SilkScreen, B.Cu at (82.5, 87.0)
- added REF**: KiCad-Logo2_20mm_SilkScreen, Symbol:KiCad-Logo2_20mm_SilkScreen, B.Cu at (124.5, 80.0)
- J2: footprint footprints:GCT_USB4105-GF-A -> footprints:USB_C_Receptacle_HRO_TYPE-C-31-M-12
- moved R7 8.04 mm to (204.2, 67.3), turned to 180 degrees
- moved C2 5.53 mm to (193.6, 69.4), turned to -90 degrees
- moved J2 1.39 mm to (214.3, 70.9)
- moved R8 1.06 mm to (204.2, 78.5)
Connections:
- C2 pad 2: GND -> Net-(C2-Pad2)
- J2 pad A5: Net-(J2-CC1) -> Net-(J2-PadA5)
- J2 pad B5: Net-(J2-CC2) -> Net-(C2-Pad2)
- R7 pad 1: GND -> Net-(C2-Pad2)
- R7 pad 2: Net-(J2-CC2) -> GND
- R8 pad 1: Net-(J2-CC1) -> GND
- R8 pad 2: GND -> Net-(J2-PadA5)
Routing:
- net Net-(C2-Pad2): track 0.00 -> 20.3 mm
- net Net-(J2-PadA5): track 0.00 -> 16.2 mm
- net Net-(J2-CC1): track 8.47 -> 0.00 mm
- net Net-(D4-K): track 0.00 -> 8.41 mm
- net Net-(J2-CC2): track 7.84 -> 0.00 mm
- net Net-(D5-K): track 4.23 -> 0.00 mm
- net +5V: track 317.9 -> 314.9 mm

Commit message: Adjusted some copper tracks. Made all resistors horizontal. Added 1K network resistor for LCD data lines. Updated version number to 1.0a and date to 3/15/2024.
Parts:
- added RN2: 1KΩ, footprints:R_Array_SIP9, F.Cu at (112.4, 48.3)
- moved R6 7.26 mm to (202.6, 83.8), turned to 0 degrees
- moved R9 6.84 mm to (156.2, 120.7), turned to 180 degrees
- moved SW2 4.41 mm to (162.6, 120.5)
- moved C1 3.27 mm to (152.9, 113.3)
- moved R2 3.27 mm to (165.1, 113.3)
- moved R3 2.14 mm to (116.8, 114.9)
- moved D6 1.41 mm to (196.8, 104.8)
- moved D2 0.64 mm to (142.9, 121.3)
Routing:
- net Net-(R2-Pad1): track 31.2 -> 23.0 mm
- net /D1: track 130.6 -> 134.6 mm
- net /D4: track 119.5 -> 123.4 mm
- net /D3: track 123.3 -> 127.2 mm
- net /D7: track 108.4 -> 112.3 mm
- net /D6: track 112.2 -> 116.2 mm
- net /D5: track 115.9 -> 119.8 mm
- net /D2: track 126.9 -> 130.8 mm
- net /D0: track 133.2 -> 137.1 mm
- net Net-(D4-K): track 8.41 -> 4.96 mm
- net +5V: track 314.9 -> 311.6 mm
- net /E: track 90.7 -> 94.0 mm
- net Net-(D2-A): track 6.02 -> 3.45 mm
- net /RS: track 104.5 -> 106.4 mm
- net /RW: track 151.5 -> 152.5 mm
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Other:
- board text added: "${project_name} Inspired by Ian Ward's YouTube Video: HD44780 Tutorial (https://www.youtube.com/watch?v=Gd6GUsHL4FI) PCB designed by an appreciative subscriber to his channel. Revision: ${version} 3/15/2024"
- board text removed: "${project_name} Inspired by Ian Ward's YouTube Video: HD44780 Tutorial (https://www.youtube.com/watch?v=Gd6GUsHL4FI) PCB designed by an appreciative subscriber to his channel. Revision: ${version} 3/6/2024"
