File: hd44780_tutorial.kicad_pcb (KiCad board)
At the start: 2 copper layers, 157.2 x 83.5 mm, 33 parts, among them J1 LCD_2004_PinSocket_1x16_P2.54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, J2 UJC-HP-3-SMT-TR, SW1 REG SELECT, SW2 ENABLE, SW3 DS02C-254-1L-08BE

Commit message: Changed project footprint/symbols directory paths from footprints/hd44780_tutorial to HD44780-tutorial-PCB/HD44780-tutorial-PCB.
Parts:
- D3: footprint footprints:LED_Bar_Graph_8_SEG_SOCKET -> HD44780-tutorial-PCB:LED_Bar_Graph_8_SEG_SOCKET
- G***: footprint footprints:Lutzcraft_logo_1125DPI -> HD44780-tutorial-PCB:Lutzcraft_logo_1125DPI
- J1: footprint footprints:LCD_2004_PinSocket_1x16_P2.54mm_Vertical -> HD44780-tutorial-PCB:LCD_2004_PinSocket_1x16_P2.54mm_Vertical
- J2: value UJC-HP-3-SMT-TR -> UJC-HP-M-G-5-MSMT-TR; footprint footprints:CUI_UJC-HP-M-G-5-MSMT-TR -> HD44780-tutorial-PCB:CUI_UJC-HP-M-G-5-MSMT-TR
- RN1, RN2: footprint footprints:R_Array_SIP9 -> HD44780-tutorial-PCB:R_Array_SIP9
- RV1, RV2: footprint footprints:BOURNE-3386P -> HD44780-tutorial-PCB:BOURNE-3386P
- S1: footprint footprints:TL2230EEF140 -> HD44780-tutorial-PCB:TL2230EEF140
- SW1, SW2: footprint footprints:SW_1825967-1 -> HD44780-tutorial-PCB:SW_1825967-1
- SW3: footprint footprints:SW_DS02C-254-1L-08BE -> HD44780-tutorial-PCB:SW_DS02C-254-1L-08BE
Changed lines of the file:
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@@
   (net 37 "unconnected-(RV1-Pad1)")
   (net 38 "unconnected-(RV2-Pad1)")
-  (footprint "footprints:SW_1825967-1" (layer "F.Cu")
+  (footprint "HD44780-tutorial-PCB:SW_1825967-1" (layer "F.Cu")
     (at 131.445 120.305)
     (property "Comment" "1825967-1")
@@
     )
   )
-  (footprint "footprints:BOURNE-3386P" (layer "F.Cu")
+  (footprint "HD44780-tutorial-PCB:BOURNE-3386P" (layer "F.Cu")
     (at 81.28 118.745)
     (tags "3386P-1-103LF ")
@@
     )
   )
-  (footprint "footprints:R_Array_SIP9" (layer "F.Cu")
+  (footprint "HD44780-tutorial-PCB:R_Array_SIP9" (layer "F.Cu")
     (at 112.395 48.26 180)
     (descr "9-pin Resistor SIP pack")
@@
     )
   )
-  (footprint "footprints:LCD_2004_PinSocket_1x16_P2.54mm_Vertical" (layer "F.Cu")
+  (footprint "HD44780-tutorial-PCB:LCD_2004_PinSocket_1x16_P2.54mm_Vertical" (layer "F.Cu")
     (at 76.9366 52.1716 90)
     (descr "Through hole straight socket strip, 1x16, 2.54mm pitch, single row (from Kicad 4.0.7), script generated")
@@
     )
   )
-  (footprint "footprints:SW_1825967-1" (layer "F.Cu")
+  (footprint "HD44780-tutorial-PCB:SW_1825967-1" (layer "F.Cu")
     (at 162.56 120.49)
     (property "Comment" "1825967-1")
@@
     )
   )
-  (footprint "footprints:CUI_UJC-HP-M-G-5-MSMT-TR" (layer "F.Cu")
+  (footprint "HD44780-tutorial-PCB:CUI_UJC-HP-M-G-5-MSMT-TR" (layer "F.Cu")
     (at 211.836 71.245 90)
     (property "MANUFACTURER" "CUI Devices")
@@
         (effects (font (size 0.8 0.787402) (thickness 0.15)))
     )
-    (fp_text value "UJC-HP-3-SMT-TR" (at 1.524 -2 90) (layer "F.Fab")
+    (fp_text value "UJC-HP-M-G-5-MSMT-TR" (at 1.524 -2 90) (layer "F.Fab")
         (effects (font (size 0.787402 0.787402) (thickness 0.15)))
     )
@@
     (pad "" np_thru_hole circle locked (at 0 0) (size 2.7 2.7) (drill 2.7) (layers "*.Cu" "*.Mask"))
   )
-  (footprint "footprints:LED_Bar_Graph_8_SEG_SOCKET" (layer "F.Cu")
+  (footprint "HD44780-tutorial-PCB:LED_Bar_Graph_8_SEG_SOCKET" (layer "F.Cu")
     (at 174.7314 94.6448 90)
     (property "Description" "LED BAR GRAPH 8-SEGMENT")
@@
     (pad "" np_thru_hole circle locked (at 0 0) (size 2.7 2.7) (drill 2.7) (layers "*.Cu" "*.Mask"))
   )
-  (footprint "footprints:BOURNE-3386P" (layer "F.Cu")
+  (footprint "HD44780-tutorial-PCB:BOURNE-3386P" (layer "F.Cu")
     (at 93.98 118.745)
     (tags "3386P-1-103LF ")
@@
     (pad "" np_thru_hole circle locked (at 0 0) (size 2.7 2.7) (drill 2.7) (layers "*.Cu" "*.Mask"))
   )
-  (footprint "footprints:SW_DS02C-254-1L-08BE" (layer "F.Cu")
+  (footprint "HD44780-tutorial-PCB:SW_DS02C-254-1L-08BE" (layer "F.Cu")
     (at 183.515 113.665)
     (property "MANUFACTURER" "CUI Inc.")
@@
     )
   )
-  (footprint "footprints:R_Array_SIP9" (layer "F.Cu")
+  (footprint "HD44780-tutorial-PCB:R_Array_SIP9" (layer "F.Cu")
     (at 172.1746 83.1644)
     (descr "9-pin Resistor SIP pack")
@@
     )
   )
-  (footprint "footprints:TL2230EEF140" (layer "F.Cu")
+  (footprint "HD44780-tutorial-PCB:TL2230EEF140" (layer "F.Cu")
     (at 206.32 105.2)
     (descr "TL2230OAF140-1")
@@
     )
   )
-  (footprint "footprints:Lutzcraft_logo_1125DPI" (layer "B.Cu")
+  (footprint "HD44780-tutorial-PCB:Lutzcraft_logo_1125DPI" (layer "B.Cu")
     (at 81.915 73.66 180)
     (attr board_only exclude_from_bom allow_missing_courtyard)

Commit message: First Kicad v8 version.
Parts:
- renumbered locked to H4

Commit message: Minor edits
Parts:
- J2: value UJC-HP-M-G-5-MSMT-TR -> USB RECEPTACLE
Changed lines of the file:
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@@
 			)
 		)
-		(property "Value" "UJC-HP-M-G-5-MSMT-TR"
-			(at 1.524 -2 90)
-			(layer "F.Fab")
+		(property "Value" "USB RECEPTACLE"
+			(at -0.0528 -1.8796 90)
+			(layer "F.SilkS")
 			(effects
 				(font
-					(size 0.787402 0.787402)
+					(size 0.8 0.7)
 					(thickness 0.15)
 				)
