File: hd44780_tutorial.kicad_sch (KiCad schematic)
At the start: 30 parts, among them J1 LCD_2004_PinSocket_1x16_P2.54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, J2 UJC-HP-3-SMT-TR, SW1 REG SELECT, SW2 ENABLE, SW3 DS02C-254-1L-08BE

Commit message: Moved footprint/model for USB-C connector to local library. Updated BOM. Updated images. Regenerated gerber/drill files.
Parts:
- J2: footprint Lutzcraft:CUI_UJC-HP-3-SMT-TR -> footprints:CUI_UJC-HP-3-SMT-TR; symbol Lutzcraft:UJC-HP-3-SMT-TR -> hd44780_tutorial:UJC-HP-3-SMT-TR
Changed lines of the file:
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@@
     )
   )
-  (symbol (lib_id "Lutzcraft:UJC-HP-3-SMT-TR") (at 238.76 42.545 0) (unit 1)
+  (symbol (lib_id "hd44780_tutorial:UJC-HP-3-SMT-TR") (at 238.76 42.545 0) (unit 1)
     (in_bom yes) (on_board yes) (dnp no)
     (property "Reference" "J2" (at 231.14 33.655 0)
@@
       (effects (font (size 1.27 1.27)) (justify left))
     )
-    (property "Footprint" "Lutzcraft:CUI_UJC-HP-3-SMT-TR" (at 238.76 42.545 0)
+    (property "Footprint" "footprints:CUI_UJC-HP-3-SMT-TR" (at 238.76 42.545 0)
       (effects (font (size 1.27 1.27)) (justify bottom) hide)
     )

Commit message: Change name and value of USB footprint to be correct.
Parts:
- J2: value UJC-HP-3-SMT-TR -> UJC-HP-M-G-5-MSMT-TR; footprint footprints:CUI_UJC-HP-3-SMT-TR -> footprints:CUI_UJC-HP-M-G-5-MSMT-TR; symbol hd44780_tutorial:UJC-HP-3-SMT-TR -> hd44780_tutorial:UJC-HP-M-G-5-MSMT-TR
Changed lines of the file:
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@@
     )
   )
-  (symbol (lib_id "hd44780_tutorial:UJC-HP-3-SMT-TR") (at 238.76 42.545 0) (unit 1)
+  (symbol (lib_id "hd44780_tutorial:UJC-HP-M-G-5-MSMT-TR") (at 238.76 42.545 0) (unit 1)
     (in_bom yes) (on_board yes) (dnp no)
     (property "Reference" "J2" (at 231.14 33.655 0)
       (effects (font (size 1.27 1.27)) (justify left))
     )
-    (property "Value" "UJC-HP-3-SMT-TR" (at 248.285 60.325 90)
+    (property "Value" "UJC-HP-M-G-5-MSMT-TR" (at 248.285 62.865 90)
       (effects (font (size 1.27 1.27)) (justify left))
     )
-    (property "Footprint" "footprints:CUI_UJC-HP-3-SMT-TR" (at 238.76 42.545 0)
+    (property "Footprint" "footprints:CUI_UJC-HP-M-G-5-MSMT-TR" (at 238.76 42.545 0)
       (effects (font (size 1.27 1.27)) (justify bottom) hide)
     )

Commit message: Changed project footprint/symbols directory paths from footprints/hd44780_tutorial to HD44780-tutorial-PCB/HD44780-tutorial-PCB.
Parts:
- D3: footprint footprints:LED_Bar_Graph_8_SEG_SOCKET -> HD44780-tutorial-PCB:LED_Bar_Graph_8_SEG_SOCKET
- J1: footprint footprints:LCD_2004_PinSocket_1x16_P2.54mm_Vertical -> HD44780-tutorial-PCB:LCD_2004_PinSocket_1x16_P2.54mm_Vertical
- J2: footprint footprints:CUI_UJC-HP-M-G-5-MSMT-TR -> HD44780-tutorial-PCB:CUI_UJC-HP-M-G-5-MSMT-TR
- RN1, RN2: footprint footprints:R_Array_SIP9 -> HD44780-tutorial-PCB:R_Array_SIP9
- RV1, RV2: footprint footprints:BOURNE-3386P -> HD44780-tutorial-PCB:BOURNE-3386P
- S1: footprint footprints:TL2230EEF140 -> HD44780-tutorial-PCB:TL2230EEF140
- SW1, SW2: footprint footprints:SW_1825967-1 -> HD44780-tutorial-PCB:SW_1825967-1
- SW3: footprint footprints:SW_DS02C-254-1L-08BE -> HD44780-tutorial-PCB:SW_DS02C-254-1L-08BE
Changed lines of the file:
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@@
       (effects (font (size 1 1)))
     )
-    (property "Footprint" "footprints:BOURNE-3386P" (at 29.21 46.99 0)
+    (property "Footprint" "HD44780-tutorial-PCB:BOURNE-3386P" (at 29.21 46.99 0)
       (effects (font (size 1 1) italic) hide)
     )
@@
       (effects (font (size 1 1)))
     )
-    (property "Footprint" "footprints:SW_1825967-1" (at 208.915 107.315 0)
+    (property "Footprint" "HD44780-tutorial-PCB:SW_1825967-1" (at 208.915 107.315 0)
       (effects (font (size 1 1)) (justify left bottom) hide)
     )
@@
       (effects (font (size 1 1)))
     )
-    (property "Footprint" "footprints:BOURNE-3386P" (at 29.21 30.48 0)
+    (property "Footprint" "HD44780-tutorial-PCB:BOURNE-3386P" (at 29.21 30.48 0)
       (effects (font (size 1 1) italic) hide)
     )
@@
       (effects (font (size 1 1)) (justify left))
     )
-    (property "Footprint" "footprints:LCD_2004_PinSocket_1x16_P2.54mm_Vertical" (at 86.995 110.49 0)
+    (property "Footprint" "HD44780-tutorial-PCB:LCD_2004_PinSocket_1x16_P2.54mm_Vertical" (at 86.995 110.49 0)
       (effects (font (size 1 1)) hide)
     )
@@
       (effects (font (size 1 1)) (justify left))
     )
-    (property "Footprint" "footprints:R_Array_SIP9" (at 146.685 62.865 90)
+    (property "Footprint" "HD44780-tutorial-PCB:R_Array_SIP9" (at 146.685 62.865 90)
       (effects (font (size 1 1)) hide)
     )
@@
       (effects (font (size 1 1)) (justify right))
     )
-    (property "Footprint" "footprints:LED_Bar_Graph_8_SEG_SOCKET" (at 119.38 73.025 0)
+    (property "Footprint" "HD44780-tutorial-PCB:LED_Bar_Graph_8_SEG_SOCKET" (at 119.38 73.025 0)
       (effects (font (size 1 1)) (justify left) hide)
     )
@@
       (effects (font (size 1 1)))
     )
-    (property "Footprint" "footprints:SW_1825967-1" (at 50.165 80.01 0)
+    (property "Footprint" "HD44780-tutorial-PCB:SW_1825967-1" (at 50.165 80.01 0)
       (effects (font (size 1 1)) (justify left bottom) hide)
     )
@@
       (effects (font (size 1.27 1.27)) (justify right))
     )
-    (property "Footprint" "footprints:SW_DS02C-254-1L-08BE" (at 133.35 111.125 0)
+    (property "Footprint" "HD44780-tutorial-PCB:SW_DS02C-254-1L-08BE" (at 133.35 111.125 0)
       (effects (font (size 1.27 1.27)) (justify left bottom) hide)
     )
@@
       (effects (font (size 1 1)))
     )
-    (property "Footprint" "footprints:TL2230EEF140" (at 146.05 232.715 0)
+    (property "Footprint" "HD44780-tutorial-PCB:TL2230EEF140" (at 146.05 232.715 0)
       (effects (font (size 1 1)) (justify left top) hide)
     )
@@
       (effects (font (size 1 1)) (justify left))
     )
-    (property "Footprint" "footprints:R_Array_SIP9" (at 60.325 102.235 90)
+    (property "Footprint" "HD44780-tutorial-PCB:R_Array_SIP9" (at 60.325 102.235 90)
       (effects (font (size 1 1)) hide)
     )
@@
       (effects (font (size 1.27 1.27)) (justify left))
     )
-    (property "Footprint" "footprints:CUI_UJC-HP-M-G-5-MSMT-TR" (at 238.76 42.545 0)
+    (property "Footprint" "HD44780-tutorial-PCB:CUI_UJC-HP-M-G-5-MSMT-TR" (at 238.76 42.545 0)
       (effects (font (size 1.27 1.27)) (justify bottom) hide)
     )

Commit message: First Kicad v8 version.
Parts:
- D3: value 8_SEG_LED BAR_GRAPH -> 8_SEG_LED BAR_GRAPH; symbol hd44780_tutorial:LED_BAR_GRAPH_8_SEG_SOCKET -> HD44780-tutorial-PCB:LED_BAR_GRAPH_8_SEG_SOCKET
- J1: symbol hd44780_tutorial:LCD_2004_PinSocket_1x16_P2.54mm_Vertical -> HD44780-tutorial-PCB:LCD_2004_PinSocket_1x16_P2.54mm_Vertical
- J2: symbol hd44780_tutorial:UJC-HP-M-G-5-MSMT-TR -> HD44780-tutorial-PCB:UJC-HP-M-G-5-MSMT-TR
- RN1, RN2: symbol hd44780_tutorial:R_Network08 -> HD44780-tutorial-PCB:R_Network08
- RV1, RV2: symbol hd44780_tutorial:BOURNE-3386P-1-502LF -> HD44780-tutorial-PCB:BOURNE-3386P-1-502LF
- S1: symbol hd44780_tutorial:TL2230EEF140 -> HD44780-tutorial-PCB:TL2230EEF140
- SW1, SW2: symbol hd44780_tutorial:SW-1825967-1 -> HD44780-tutorial-PCB:SW-1825967-1
- SW3: symbol hd44780_tutorial:DS02C-254-1L-08BE -> HD44780-tutorial-PCB:DS02C-254-1L-08BE
